Commit message: 添加了光学平台,将平台的urdf文件加入到了机械臂代码中，但是在轨迹规划时需要加入平台的碰撞模型,并发布到rviz2中.

File: src/mybot_description/urdf/assumble.urdf.xacro (robot description, xacro)
@@ -8,6 +8,6 @@
   <joint name="table_to_world" type="fixed">
     <parent link="world"/>
-    <child link="box"/>
-    <origin rpy="0 0 0" xyz="0 0.3 0"/>   <!-- 桌子位于世界原点，可根据需要调整 -->
+    <child link="table_link"/>
+    <origin rpy="0 0 0" xyz="0 0 0"/>   <!-- 桌子位于世界原点，可根据需要调整 -->
   </joint>
 </robot>

File: src/mybot_description/urdf/ur7e.urdf.xacro (robot description, xacro)
@@ -52,4 +52,11 @@
   -->
   <!-- create link fixed to the "world" -->
+  <xacro:include filename="$(find optical_platform_description)/urdf/optical_platform_description.urdf" />
+  <!-- ========== 固定关节：将桌子固定到世界坐标系 ========== -->
+  <joint name="table_to_world" type="fixed">
+    <parent link="world"/>
+    <child link="table_base_link"/>   <!-- 注意：桌子的 root link 名称必须与此一致 -->
+    <origin xyz="0.0 0.0 0.8" rpy="0 0 0"/>
+  </joint>
   <link name="world"/>
   <link name="ground_plane">
@@ -291,5 +298,5 @@
   <!-- base_joint fixes base_link to the environment -->
   <joint name="base_joint" type="fixed">
-    <origin rpy="0 0 0" xyz="0 0 0"/>
+    <origin rpy="0 0 0" xyz="-0.4 -0.4 0.8"/>
     <parent link="world"/>
     <child link="base_link"/>
@@ -399,5 +406,5 @@
   <xacro:include filename="$(find realsense2_description)/urdf/_d435i.urdf.xacro" />
   <xacro:sensor_d435i parent="world" name="camera" use_nominal_extrinsics="true">
-      <origin xyz="0.4 0 1.2" rpy="0 1.5708 0"/>
+      <origin xyz="0.4 0 2.2" rpy="0 1.5708 0"/>
   </xacro:sensor_d435i>
   <gazebo reference="camera_link">
