Commit message: 修复了圆柱点云在rviz和gazebo中不相匹配

File: src/mybot_description/urdf/ur7e.urdf.xacro (robot description, xacro)
@@ -399,5 +399,5 @@
   <xacro:include filename="$(find realsense2_description)/urdf/_d435i.urdf.xacro" />
   <xacro:sensor_d435i parent="world" name="camera" use_nominal_extrinsics="true">
-      <origin xyz="0.2 0 1.2" rpy="0 1.5708 0"/>
+      <origin xyz="0.4 0 1.2" rpy="0 1.5708 0"/>
   </xacro:sensor_d435i>
   <gazebo reference="camera_link">

Commit message: 重新配置了实验环境的moveit包,且可以正常使用

File: src/mybot_description/urdf/ur7e.urdf.xacro (robot description, xacro)
@@ -66,5 +66,5 @@
       <origin rpy="0 0 0" xyz="0 0 0"/>
       <geometry>
-        <box size="5 5 0"/>
+        <box size="5 5 0.01"/>
       </geometry>
       <material name="ground_white">
@@ -73,15 +73,16 @@
     </visual>
     <collision>
-      <origin rpy="0 0 0" xyz="0 0 0"/>
-      <geometry>
-        <box size="5 5 0"/>
+      <origin rpy="0 0 0" xyz="0 0 -0.005"/>
+      <geometry>
+        <box size="5 5 0.01"/>
       </geometry>
     </collision>
   </link>
   <joint name="ground_plane_joint" type="fixed">
-    <origin rpy="0 0 0" xyz="0 0 -0.01"/>
+    <origin rpy="0 0 0" xyz="0 0 -0.005"/>
     <parent link="world"/>
     <child link="ground_plane"/>
   </joint>
+  <!-- ros2_control 代码起始 -->
   <ros2_control name="ur7e" type="system">
     <hardware>
@@ -159,4 +160,5 @@
     </joint>
   </ros2_control>
+  <!-- ros2_control 代码结束 -->
   <!-- Add URDF transmission elements (for ros_control) -->
   <!--<xacro:ur_arm_transmission prefix="${prefix}" hw_interface="${transmission_hw_interface}" />-->

File: src/ur7e_moveit_config/config/ur7e.ros2_control.xacro (robot description, xacro)
@@ -14,4 +14,5 @@
                 </state_interface>
                 <state_interface name="velocity"/>
+                <state_interface name="effort"/>
             </joint>
             <joint name="shoulder_lift_joint">
@@ -21,4 +22,5 @@
                 </state_interface>
                 <state_interface name="velocity"/>
+                <state_interface name="effort"/>
             </joint>
             <joint name="elbow_joint">
@@ -28,4 +30,5 @@
                 </state_interface>
                 <state_interface name="velocity"/>
+                <state_interface name="effort"/>
             </joint>
             <joint name="wrist_1_joint">
@@ -35,4 +38,5 @@
                 </state_interface>
                 <state_interface name="velocity"/>
+                <state_interface name="effort"/>
             </joint>
             <joint name="wrist_2_joint">
@@ -42,4 +46,5 @@
                 </state_interface>
                 <state_interface name="velocity"/>
+                <state_interface name="effort"/>
             </joint>
             <joint name="wrist_3_joint">
@@ -49,4 +54,5 @@
                 </state_interface>
                 <state_interface name="velocity"/>
+                <state_interface name="effort"/>
             </joint>
         </ros2_control>

Commit message: 添加了ft300六维力传感器,增加了接收力矩的功能,使用ros2 topic echo /robotiq_ft300/ft_sensor_wrench,订阅力矩信息

File: src/mybot_description/urdf/ur7e.urdf.xacro (robot description, xacro)
@@ -1,65 +1,13 @@
 <?xml version="1.0" ?>
-<!-- =================================================================================== -->
-<!-- |    This document was autogenerated by xacro from /opt/ros/humble/share/ur_description/urdf/ur.urdf.xacro | -->
-<!-- |    EDITING THIS FILE BY HAND IS NOT RECOMMENDED                                 | -->
-<!-- =================================================================================== -->
 <robot name="ur7e" xmlns:xacro="http://ros.org/wiki/xacro">
-  <!--
-    Base UR robot series xacro macro.
-    NOTE this is NOT a URDF. It cannot directly be loaded by consumers
-    expecting a flattened '.urdf' file. See the top-level '.xacro' for that
-    (but note that .xacro must still be processed by the xacro command).
-    This file models the base kinematic chain of a UR robot, which then gets
-    parameterised by various configuration files to convert it into a UR3(e),
-    UR5(e), UR10(e) or UR16e, etc.
-    NOTE the default kinematic parameters (i.e., link lengths, frame locations,
-    offsets, etc) do not correspond to any particular robot. They are defaults
-    only. There WILL be non-zero offsets between the Forward Kinematics results
-    in TF (i.e., robot_state_publisher) and the values reported by the Teach
-    Pendant.
-    For accurate (and robot-specific) transforms, the 'kinematics_parameters_file'
-    parameter MUST point to a .yaml file containing the appropriate values for
-    the targeted robot.
-    If using the UniversalRobots/Universal_Robots_ROS_Driver, follow the steps
-    described in the readme of that repository to extract the kinematic
-    calibration from the controller and generate the required .yaml file.
-    Main author of the migration to yaml configs Ludovic Delval.
-    Contributors to previous versions (in no particular order)
-     - Denis Stogl
-     - Lovro Ivanov
-     - Felix Messmer
-     - Kelsey Hawkins
-     - Wim Meeussen
-     - Shaun Edwards
-     - Nadia Hammoudeh Garcia
-     - Dave Hershberger
-     - G. vd. Hoorn
-     - Philip Long
-     - Dave Coleman
-     - Miguel Prada
-     - Mathias Luedtke
-     - Marcel Schnirring
-     - Felix von Drigalski
-     - Felix Exner
-     - Jimmy Da Silva
-     - Ajit Krisshna N L
-     - Muhammad Asif Rana
-  -->
-  <!--
-    NOTE the macro defined in this file is NOT part of the public API of this
-          package. Users CANNOT rely on this file being available, or stored in
-          this location. Nor can they rely on the existence of the macro.
-  -->
-  <!-- create link fixed to the "world" -->
   <xacro:include filename="$(find optical_platiform_description)/urdf/optical_platiform_description.urdf" />
   <xacro:include filename="$(find robot_arm_base_link)/urdf/robot_arm_base_link.urdf" />
   <xacro:include filename="$(find sensers_fixture_description)/urdf/sensers_fixture_description.urdf" />
-  <!-- ========== 固定关节：将桌子固定到世界坐标系 ========== -->
+  <link name="world"/>
   <joint name="table_to_world" type="fixed">
     <parent link="world"/>
-    <child link="optical_platiform_base_link"/>   <!-- 注意：桌子的 root link 名称必须与此一致 -->
+    <child link="optical_platiform_base_link"/>
     <origin xyz="0.0 0.0 0.8" rpy="0 0 0"/>
   </joint>
-  <link name="world"/>
   <link name="ground_plane">
     <visual>
@@ -84,5 +32,5 @@
     <child link="ground_plane"/>
   </joint>
-  <!-- ros2_control 代码起始 -->
+<!-- ros2_control开始地方 -->
   <ros2_control name="ur7e" type="system">
     <hardware>
@@ -98,5 +46,4 @@
       <command_interface name="effort"/>
       <state_interface name="position">
-        <!-- initial position for the FakeSystem and simulation -->
         <param name="initial_value">0.0</param>
       </state_interface>
@@ -109,5 +56,4 @@
       <command_interface name="effort"/>
       <state_interface name="position">
-        <!-- initial position for the FakeSystem and simulation -->
         <param name="initial_value">-1.57</param>
       </state_interface>
@@ -120,5 +66,4 @@
       <command_interface name="effort"/>
       <state_interface name="position">
-        <!-- initial position for the FakeSystem and simulation -->
         <param name="initial_value">0.0</param>
       </state_interface>
@@ -131,5 +76,4 @@
       <command_interface name="effort"/>
       <state_interface name="position">
-        <!-- initial position for the FakeSystem and simulation -->
         <param name="initial_value">-1.57</param>
       </state_interface>
@@ -142,5 +86,4 @@
       <command_interface name="effort"/>
       <state_interface name="position">
-        <!-- initial position for the FakeSystem and simulation -->
         <param name="initial_value">0.0</param>
       </state_interface>
@@ -153,5 +96,4 @@
       <command_interface name="effort"/>
       <state_interface name="position">
-        <!-- initial position for the FakeSystem and simulation -->
         <param name="initial_value">0.0</param>
       </state_interface>
@@ -159,10 +101,11 @@
       <state_interface name="effort"/>
     </joint>
+    <joint name="ft300_sensor_joint">
+      <state_interface name="position">
+        <param name="initial_value">0.0</param>
+      </state_interface>
+    </joint>
   </ros2_control>
-  <!-- ros2_control 代码结束 -->
-  <!-- Add URDF transmission elements (for ros_control) -->
-  <!--<xacro:ur_arm_transmission prefix="${prefix}" hw_interface="${transmission_hw_interface}" />-->
-  <!-- Placeholder for ros2_control transmission which don't yet exist -->
-  <!-- links -  main serial chain -->
+<!-- ros2_control结束地方 -->
   <link name="base_link"/>
   <link name="base_link_inertia">
@@ -170,5 +113,5 @@
       <origin rpy="0 0 3.141592653589793" xyz="0 0 0"/>
       <geometry>
-        <mesh filename="file:///opt/ros/humble/share/ur_description/meshes/ur5e/visual/base.dae"/>
+         <mesh filename="file:///opt/ros/humble/share/ur_description/meshes/ur5e/visual/base.dae"/>
       </geometry>
     </visual>
@@ -231,5 +174,5 @@
     </visual>
     <collision>
-      <origin rpy="1.5707963267948966 0 -1.5707963267948966" xyz="0 0 0.007"/>
+       <origin rpy="1.5707963267948966 0 -1.5707963267948966" xyz="0 0 0.007"/>
       <geometry>
         <mesh filename="file:///opt/ros/humble/share/ur_description/meshes/ur5e/collision/forearm.stl"/>
@@ -299,28 +242,17 @@
     </inertial>
   </link>
-  <!--改变机械臂在仿真环境中的位置-->
-  <!-- base_joint fixes base_link to the environment -->
-  <!-- 2. 机械臂底座固定在光学平台上 -->
   <joint name="base_to_table" type="fixed">
     <parent link="optical_platiform_base_link"/>
-    <child link="robot_arm_base_link"/>   <!-- 底座的 link -->
+    <child link="robot_arm_base_link"/>
     <origin xyz="-0.325 -0.625 0.0" rpy="0 0 0"/>
   </joint>
-  <!-- 3. 机械臂的 base_link 固定在底座上（原 base_joint 需修改） -->
-  <!-- 注意：删除原来的 base_joint，使用以下定义 -->
   <joint name="base_joint" type="fixed">
     <parent link="robot_arm_base_link"/>
-    <child link="base_link"/>            <!-- UR7e 的基座 link -->
-    <origin xyz="-0.0 0.0 0.025" rpy="0 0 0"/>  <!-- 偏移量根据实际调整 -->
-  </joint>
-  <!-- joints - main serial chain -->
+    <child link="base_link"/>
+    <origin xyz="-0.0 0.0 0.025" rpy="0 0 0"/>
+  </joint>
   <joint name="base_link-base_link_inertia" type="fixed">
     <parent link="base_link"/>
     <child link="base_link_inertia"/>
-    <!-- 'base_link' is REP-103 aligned (so X+ forward), while the internal
-           frames of the robot/controller have X+ pointing backwards.
-           Use the joint between 'base_link' and 'base_link_inertia' (a dummy
-           link/frame) to introduce the necessary rotation over Z (of pi rad).
-      -->
     <origin rpy="0 0 3.141592653589793" xyz="0 0 0"/>
   </joint>
@@ -379,17 +311,10 @@
     <origin rpy="3.141592653589793 0 0" xyz="0 0 0"/>
   </joint>
-  <!-- ROS-Industrial 'base' frame - base_link to UR 'Base' Coordinates transform -->
   <link name="base"/>
   <joint name="base_link-base_fixed_joint" type="fixed">
-    <!-- Note the rotation over Z of pi radians - as base_link is REP-103
-           aligned (i.e., has X+ forward, Y+ left and Z+ up), this is needed
-           to correctly align 'base' with the 'Base' coordinate system of
-           the UR controller.
-      -->
     <origin rpy="0 0 3.141592653589793" xyz="0 0 0"/>
     <parent link="base_link"/>
     <child link="base"/>
   </joint>
-  <!-- ROS-Industrial 'flange' frame - attachment point for EEF models -->
   <link name="flange"/>
   <joint name="wrist_3-flange" type="fixed">
@@ -398,27 +323,104 @@
     <origin rpy="0 -1.5707963267948966 -1.5707963267948966" xyz="0 0 0"/>
   </joint>
-  <!-- ROS-Industrial 'tool0' frame - all-zeros tool frame -->
   <link name="tool0"/>
   <joint name="flange-tool0" type="fixed">
-    <!-- default toolframe - X+ left, Y+ up, Z+ front -->
     <origin rpy="1.5707963267948966 0 1.5707963267948966" xyz="0 0 0"/>
     <parent link="flange"/>
     <child link="tool0"/>
   </joint>
-    <!-- 将夹具固定在 tool0 上 -->
+  <joint name="ft300_fix" type="fixed">
+    <origin rpy="0 0 0" xyz="0 0 0"/>
+    <parent link="tool0"/>
+    <child link="ft300_mounting_plate"/>
+  </joint>
+  <link name="ft300_mounting_plate">
+    <visual>
+      <origin rpy="0 0 0" xyz="0 0 0"/>
+      <geometry>
+        <mesh filename="file:///home/lk/ur_sim/install/mybot_description/share/mybot_description/meshes/visual/mountings/robotiq_ft300-G-062-COUPLING_G-50-4M6-1D6_20181119.STL"/>
+      </geometry>
+      <material name="Robotiq-Grey">
+        <color rgba="0.4 0.4 0.4 1.0"/>
+      </material>
+    </visual>
+    <collision>
+      <origin rpy="0 0 0" xyz="0 0 0"/>
+      <geometry>
+        <mesh filename="file:///home/lk/ur_sim/install/mybot_description/share/mybot_description/meshes/collision/mountings/robotiq_ft300-G-062-COUPLING_G-50-4M6-1D6_20181119.STL"/>
+      </geometry>
+    </collision>
+  </link>
+  <joint name="ft300_mounting_plate_joint" type="fixed">
+    <origin rpy="0 3.141592653589793 0" xyz="0 0 0.0415"/>
+    <parent link="ft300_mounting_plate"/>
+    <child link="ft300_sensor"/>
+  </joint>
+  <link name="ft300_sensor">
+    <inertial>
+      <origin rpy="0 0 0" xyz="0 0 -0.017"/>
+      <mass value="0.300"/>
+      <inertia ixx="0.000262" ixy="0" ixz="1e-06" iyx="0" iyy="0.000265" iyz="1e-06" izx="-1e-06" izy="1e-06" izz="0.000219"/>
+    </inertial>
+    <visual>
+      <origin rpy="0 0 0" xyz="0 0 0"/>
+      <geometry>
+        <mesh filename="file:///home/lk/ur_sim/install/mybot_description/share/mybot_description/meshes/visual/robotiq_ft300.STL"/>
+      </geometry>
+      <material name="Robotiq-Black">
+        <color rgba="0.2 0.2 0.2 1.0"/>
+      </material>
+    </visual>
+    <collision>
+      <origin rpy="0 0 0" xyz="0 0 0"/>
+      <geometry>
+        <mesh filename="file:///home/lk/ur_sim/install/mybot_description/share/mybot_description/meshes/collision/robotiq_ft300.STL"/>
+      </geometry>
+    </collision>
+  </link>
+  <joint name="measurment_joint" type="fixed">
+    <origin rpy="0 3.141592653589793 -1.5707963267948966" xyz="0 0 0"/>
+    <parent link="ft300_sensor"/>
+    <child link="robotiq_ft_frame_id"/>
+  </joint>
+  <link name="robotiq_ft_frame_id"/>
+  <link name="force_transfer_link">
+    <inertial>
+      <origin rpy="0 0 0" xyz="0 0 0"/>
+      <mass value="0.01"/> <inertia ixx="1e-6" ixy="0.0" ixz="0.0" iyy="1e-6" iyz="0.0" izz="1e-6"/>
+    </inertial>
+  </link>
+  <joint name="ft300_sensor_joint" type="revolute">
+    <origin rpy="0 3.141592653589793 -1.5707963267948966" xyz="0 0 0"/>
+    <parent link="ft300_sensor"/>
+    <child link="force_transfer_link"/> <axis xyz="0 0 1"/>
+    <limit lower="0.0" upper="0.0" effort="1000.0" velocity="0.0"/>
+  </joint>
   <joint name="fixture_joint" type="fixed">
-    <parent link="tool0"/>
-    <child link="sensers_fixture"/>   <!-- 此处 fixture_link 应与夹具 URDF 中的 link 名称一致 -->
-    <origin xyz="0.0 0.0 0.0" rpy="1.5707963267948966 0 0"/>   <!-- 根据实际安装位置调整 -->
-  </joint>
-  <link name="tcp_link"/>
-  <joint name="fixture_to_tcp" type="fixed">
-    <parent link="sensers_fixture"/>
-    <child link="tcp_link"/>
-    <origin xyz="0 0 0.01" rpy="0 0 0"/>  <!-- 探头相对于夹具的偏移 -->
-  </joint>
-  <!-- Gazebo plugins -->
+    <parent link="force_transfer_link"/>
+    <child link="sensers_fixture"/>
+    <origin xyz="0.0 0.0 0.0" rpy="1.5707963267948966 0 0"/>
+  </joint>
+  <gazebo reference="ft300_sensor">
+    <material>Gazebo/DarkGrey</material>
+  </gazebo>
+  <gazebo reference="ft300_mounting_plate">
+    <material>Gazebo/Gray</material>
+  </gazebo>
+  <gazebo reference="ft300_sensor_joint">
+    <provideFeedback>true</provideFeedback>
+  </gazebo>
+  <gazebo>
+    <plugin filename="libgazebo_ros_ft_sensor.so" name="gazebo_ros_ft_sensor">
+      <ros>
+        <namespace>/robotiq_ft300</namespace>
+        <remapping>wrench:=ft_sensor_wrench</remapping>
+      </ros>
+      <joint_name>ft300_sensor_joint</joint_name>
+      <update_rate>50.0</update_rate>
+      <gaussian_noise>0.01</gaussian_noise>
+    </plugin>
+  </gazebo>
   <gazebo reference="world">
-    </gazebo>
+  </gazebo>
   <gazebo>
     <plugin filename="libgazebo_ros2_control.so" name="gazebo_ros2_control">
@@ -447,5 +449,4 @@
                   <far>2.0</far>
               </clip>
-            <!-- 新增深度相机配置 -->
             <depth_camera>
                 <image>

File: src/ur7e_moveit_config/config/ur7e.ros2_control.xacro (robot description, xacro)
@@ -14,5 +14,4 @@
                 </state_interface>
                 <state_interface name="velocity"/>
-                <state_interface name="effort"/>
             </joint>
             <joint name="shoulder_lift_joint">
@@ -22,5 +21,4 @@
                 </state_interface>
                 <state_interface name="velocity"/>
-                <state_interface name="effort"/>
             </joint>
             <joint name="elbow_joint">
@@ -30,5 +28,4 @@
                 </state_interface>
                 <state_interface name="velocity"/>
-                <state_interface name="effort"/>
             </joint>
             <joint name="wrist_1_joint">
@@ -38,5 +35,4 @@
                 </state_interface>
                 <state_interface name="velocity"/>
-                <state_interface name="effort"/>
             </joint>
             <joint name="wrist_2_joint">
@@ -46,5 +42,4 @@
                 </state_interface>
                 <state_interface name="velocity"/>
-                <state_interface name="effort"/>
             </joint>
             <joint name="wrist_3_joint">
@@ -54,5 +49,4 @@
                 </state_interface>
                 <state_interface name="velocity"/>
-                <state_interface name="effort"/>
             </joint>
         </ros2_control>
