Commit message: 添加配置了moveit servo,启动流程如下

File: src/mybot_description/urdf/ur7e.urdf.xacro (robot description, xacro)
@@ -3,5 +3,5 @@
   <xacro:include filename="$(find optical_platiform_description)/urdf/optical_platiform_description.urdf" />
   <xacro:include filename="$(find robot_arm_base_link)/urdf/robot_arm_base_link.urdf" />
-  <xacro:include filename="$(find sensers_fixture_description)/urdf/sensers_fixture_description.urdf" />
+  <xacro:include filename="$(find sensors_fixture_description)/urdf/sensors_fixture_description.urdf" />
   <link name="world"/>
   <joint name="table_to_world" type="fixed">
@@ -32,9 +32,8 @@
     <child link="ground_plane"/>
   </joint>
-<!-- ros2_control开始地方 -->
+<!-- ros2_control 开始 -->
   <ros2_control name="ur7e" type="system">
     <hardware>
       <plugin>gazebo_ros2_control/GazeboSystem</plugin>
-      <plugin>mock_components/GenericSystem</plugin>
       <param name="fake_sensor_commands">False</param>
       <param name="state_following_offset">0.0</param>
@@ -45,7 +44,5 @@
       <command_interface name="velocity"/>
       <command_interface name="effort"/>
-      <state_interface name="position">
-        <param name="initial_value">0.0</param>
-      </state_interface>
+      <state_interface name="position"><param name="initial_value">0.0</param></state_interface>
       <state_interface name="velocity"/>
       <state_interface name="effort"/>
@@ -55,7 +52,5 @@
       <command_interface name="velocity"/>
       <command_interface name="effort"/>
-      <state_interface name="position">
-        <param name="initial_value">-1.57</param>
-      </state_interface>
+      <state_interface name="position"><param name="initial_value">-1.57</param></state_interface>
       <state_interface name="velocity"/>
       <state_interface name="effort"/>
@@ -65,7 +60,5 @@
       <command_interface name="velocity"/>
       <command_interface name="effort"/>
-      <state_interface name="position">
-        <param name="initial_value">0.0</param>
-      </state_interface>
+      <state_interface name="position"><param name="initial_value">0.0</param></state_interface>
       <state_interface name="velocity"/>
       <state_interface name="effort"/>
@@ -75,7 +68,5 @@
       <command_interface name="velocity"/>
       <command_interface name="effort"/>
-      <state_interface name="position">
-        <param name="initial_value">-1.57</param>
-      </state_interface>
+      <state_interface name="position"><param name="initial_value">-1.57</param></state_interface>
       <state_interface name="velocity"/>
       <state_interface name="effort"/>
@@ -85,7 +76,5 @@
       <command_interface name="velocity"/>
       <command_interface name="effort"/>
-      <state_interface name="position">
-        <param name="initial_value">0.0</param>
-      </state_interface>
+      <state_interface name="position"><param name="initial_value">0.0</param></state_interface>
       <state_interface name="velocity"/>
       <state_interface name="effort"/>
@@ -95,30 +84,24 @@
       <command_interface name="velocity"/>
       <command_interface name="effort"/>
-      <state_interface name="position">
-        <param name="initial_value">0.0</param>
-      </state_interface>
+      <state_interface name="position"><param name="initial_value">0.0</param></state_interface>
       <state_interface name="velocity"/>
       <state_interface name="effort"/>
     </joint>
     <joint name="ft300_sensor_joint">
-      <state_interface name="position">
-        <param name="initial_value">0.0</param>
-      </state_interface>
+      <state_interface name="position"><param name="initial_value">0.0</param></state_interface>
+      <state_interface name="velocity"><param name="initial_value">0.0</param></state_interface>
+      <state_interface name="effort"><param name="initial_value">0.0</param></state_interface>
     </joint>
   </ros2_control>
-<!-- ros2_control结束地方 -->
+<!-- ros2_control 结束 -->
   <link name="base_link"/>
   <link name="base_link_inertia">
     <visual>
       <origin rpy="0 0 3.141592653589793" xyz="0 0 0"/>
-      <geometry>
-         <mesh filename="file:///opt/ros/humble/share/ur_description/meshes/ur5e/visual/base.dae"/>
-      </geometry>
+      <geometry><mesh filename="file:///opt/ros/humble/share/ur_description/meshes/ur5e/visual/base.dae"/></geometry>
     </visual>
     <collision>
       <origin rpy="0 0 3.141592653589793" xyz="0 0 0"/>
-      <geometry>
-        <mesh filename="file:///opt/ros/humble/share/ur_description/meshes/ur5e/collision/base.stl"/>
-      </geometry>
+      <geometry><mesh filename="file:///opt/ros/humble/share/ur_description/meshes/ur5e/collision/base.stl"/></geometry>
     </collision>
     <inertial>
@@ -131,13 +114,9 @@
     <visual>
       <origin rpy="0 0 3.141592653589793" xyz="0 0 0"/>
-      <geometry>
-        <mesh filename="file:///opt/ros/humble/share/ur_description/meshes/ur5e/visual/shoulder.dae"/>
-      </geometry>
+      <geometry><mesh filename="file:///opt/ros/humble/share/ur_description/meshes/ur5e/visual/shoulder.dae"/></geometry>
     </visual>
     <collision>
       <origin rpy="0 0 3.141592653589793" xyz="0 0 0"/>
-      <geometry>
-        <mesh filename="file:///opt/ros/humble/share/ur_description/meshes/ur5e/collision/shoulder.stl"/>
-      </geometry>
+      <geometry><mesh filename="file:///opt/ros/humble/share/ur_description/meshes/ur5e/collision/shoulder.stl"/></geometry>
     </collision>
     <inertial>
@@ -150,13 +129,9 @@
     <visual>
       <origin rpy="1.5707963267948966 0 -1.5707963267948966" xyz="0 0 0.138"/>
-      <geometry>
-        <mesh filename="file:///opt/ros/humble/share/ur_description/meshes/ur5e/visual/upperarm.dae"/>
-      </geometry>
+      <geometry><mesh filename="file:///opt/ros/humble/share/ur_description/meshes/ur5e/visual/upperarm.dae"/></geometry>
     </visual>
     <collision>
       <origin rpy="1.5707963267948966 0 -1.5707963267948966" xyz="0 0 0.138"/>
-      <geometry>
-        <mesh filename="file:///opt/ros/humble/share/ur_description/meshes/ur5e/collision/upperarm.stl"/>
-      </geometry>
+      <geometry><mesh filename="file:///opt/ros/humble/share/ur_description/meshes/ur5e/collision/upperarm.stl"/></geometry>
     </collision>
     <inertial>
@@ -169,13 +144,9 @@
     <visual>
       <origin rpy="1.5707963267948966 0 -1.5707963267948966" xyz="0 0 0.007"/>
-      <geometry>
-        <mesh filename="file:///opt/ros/humble/share/ur_description/meshes/ur5e/visual/forearm.dae"/>
-      </geometry>
-    </visual>
-    <collision>
-       <origin rpy="1.5707963267948966 0 -1.5707963267948966" xyz="0 0 0.007"/>
-      <geometry>
-        <mesh filename="file:///opt/ros/humble/share/ur_description/meshes/ur5e/collision/forearm.stl"/>
-      </geometry>
+      <geometry><mesh filename="file:///opt/ros/humble/share/ur_description/meshes/ur5e/visual/forearm.dae"/></geometry>
+    </visual>
+    <collision>
+      <origin rpy="1.5707963267948966 0 -1.5707963267948966" xyz="0 0 0.007"/>
+      <geometry><mesh filename="file:///opt/ros/humble/share/ur_description/meshes/ur5e/collision/forearm.stl"/></geometry>
     </collision>
     <inertial>
@@ -188,13 +159,9 @@
     <visual>
       <origin rpy="1.5707963267948966 0 0" xyz="0 0 -0.127"/>
-      <geometry>
-        <mesh filename="file:///opt/ros/humble/share/ur_description/meshes/ur5e/visual/wrist1.dae"/>
-      </geometry>
+      <geometry><mesh filename="file:///opt/ros/humble/share/ur_description/meshes/ur5e/visual/wrist1.dae"/></geometry>
     </visual>
     <collision>
       <origin rpy="1.5707963267948966 0 0" xyz="0 0 -0.127"/>
-      <geometry>
-        <mesh filename="file:///opt/ros/humble/share/ur_description/meshes/ur5e/collision/wrist1.stl"/>
-      </geometry>
+      <geometry><mesh filename="file:///opt/ros/humble/share/ur_description/meshes/ur5e/collision/wrist1.stl"/></geometry>
     </collision>
     <inertial>
@@ -207,13 +174,9 @@
     <visual>
       <origin rpy="0 0 0" xyz="0 0 -0.0997"/>
-      <geometry>
-        <mesh filename="file:///opt/ros/humble/share/ur_description/meshes/ur5e/visual/wrist2.dae"/>
-      </geometry>
+      <geometry><mesh filename="file:///opt/ros/humble/share/ur_description/meshes/ur5e/visual/wrist2.dae"/></geometry>
     </visual>
     <collision>
       <origin rpy="0 0 0" xyz="0 0 -0.0997"/>
-      <geometry>
-        <mesh filename="file:///opt/ros/humble/share/ur_description/meshes/ur5e/collision/wrist2.stl"/>
-      </geometry>
+      <geometry><mesh filename="file:///opt/ros/humble/share/ur_description/meshes/ur5e/collision/wrist2.stl"/></geometry>
     </collision>
     <inertial>
@@ -226,13 +189,9 @@
     <visual>
       <origin rpy="1.5707963267948966 0 0" xyz="0 0 -0.0989"/>
-      <geometry>
-        <mesh filename="file:///opt/ros/humble/share/ur_description/meshes/ur5e/visual/wrist3.dae"/>
-      </geometry>
+      <geometry><mesh filename="file:///opt/ros/humble/share/ur_description/meshes/ur5e/visual/wrist3.dae"/></geometry>
     </visual>
     <collision>
       <origin rpy="1.5707963267948966 0 0" xyz="0 0 -0.0989"/>
-      <geometry>
-        <mesh filename="file:///opt/ros/humble/share/ur_description/meshes/ur5e/collision/wrist3.stl"/>
-      </geometry>
+      <geometry><mesh filename="file:///opt/ros/humble/share/ur_description/meshes/ur5e/collision/wrist3.stl"/></geometry>
     </collision>
     <inertial>
@@ -340,13 +299,9 @@
         <mesh filename="file:///home/lk/ur_sim/install/mybot_description/share/mybot_description/meshes/visual/mountings/robotiq_ft300-G-062-COUPLING_G-50-4M6-1D6_20181119.STL"/>
       </geometry>
-      <material name="Robotiq-Grey">
-        <color rgba="0.4 0.4 0.4 1.0"/>
-      </material>
-    </visual>
-    <collision>
-      <origin rpy="0 0 0" xyz="0 0 0"/>
-      <geometry>
-        <mesh filename="file:///home/lk/ur_sim/install/mybot_description/share/mybot_description/meshes/collision/mountings/robotiq_ft300-G-062-COUPLING_G-50-4M6-1D6_20181119.STL"/>
-      </geometry>
+      <material name="Robotiq-Grey"><color rgba="0.4 0.4 0.4 1.0"/></material>
+    </visual>
+    <collision>
+      <origin rpy="0 0 0" xyz="0 0 0"/>
+      <geometry><mesh filename="file:///home/lk/ur_sim/install/mybot_description/share/mybot_description/meshes/collision/mountings/robotiq_ft300-G-062-COUPLING_G-50-4M6-1D6_20181119.STL"/></geometry>
     </collision>
   </link>
@@ -364,16 +319,10 @@
     <visual>
       <origin rpy="0 0 0" xyz="0 0 0"/>
-      <geometry>
-        <mesh filename="file:///home/lk/ur_sim/install/mybot_description/share/mybot_description/meshes/visual/robotiq_ft300.STL"/>
-      </geometry>
-      <material name="Robotiq-Black">
-        <color rgba="0.2 0.2 0.2 1.0"/>
-      </material>
-    </visual>
-    <collision>
-      <origin rpy="0 0 0" xyz="0 0 0"/>
-      <geometry>
-        <mesh filename="file:///home/lk/ur_sim/install/mybot_description/share/mybot_description/meshes/collision/robotiq_ft300.STL"/>
-      </geometry>
+      <geometry><mesh filename="file:///home/lk/ur_sim/install/mybot_description/share/mybot_description/meshes/visual/robotiq_ft300.STL"/></geometry>
+      <material name="Robotiq-Black"><color rgba="0.2 0.2 0.2 1.0"/></material>
+    </visual>
+    <collision>
+      <origin rpy="0 0 0" xyz="0 0 0"/>
+      <geometry><mesh filename="file:///home/lk/ur_sim/install/mybot_description/share/mybot_description/meshes/collision/robotiq_ft300.STL"/></geometry>
     </collision>
   </link>
@@ -393,11 +342,28 @@
     <origin rpy="0 3.141592653589793 -1.5707963267948966" xyz="0 0 0"/>
     <parent link="ft300_sensor"/>
-    <child link="force_transfer_link"/> <axis xyz="0 0 1"/>
+    <child link="force_transfer_link"/>
+    <axis xyz="0 0 1"/>
     <limit lower="0.0" upper="0.0" effort="1000.0" velocity="0.0"/>
   </joint>
   <joint name="fixture_joint" type="fixed">
     <parent link="force_transfer_link"/>
-    <child link="sensers_fixture"/>
-    <origin xyz="0.0 0.0 0.0" rpy="1.5707963267948966 0 0"/>
+    <child link="sensors_fixture_base_link"/>
+    <origin xyz="0.0 0.0 0.0" rpy="0 0 3.141592653589793"/>
+  </joint>
+  <xacro:include filename="$(find realsense2_description)/urdf/_d435i.urdf.xacro" />
+  <xacro:sensor_d435i parent="sensors_fixture_base_link" name="camera" use_nominal_extrinsics="true">
+      <origin xyz="0.1 0 0.0185" rpy="0 -1.5708 0"/>
+  </xacro:sensor_d435i>
+  <link name="camera_tcp_link"/>
+  <joint name="camera_tcp_joint" type="fixed">
+    <parent link="sensors_fixture_base_link"/>
+    <child link="camera_tcp_link"/>
+    <origin xyz="0.0 0 0.0" rpy="0 -1.5708 0"/>
+  </joint>
+  <link name="ultrasonic_tcp_link"/>
+  <joint name="ultrasonic_tcp_joint" type="fixed">
+    <parent link="sensors_fixture_base_link"/>
+    <child link="ultrasonic_tcp_link"/>
+    <origin xyz="0.0 0.0 0.12" rpy="0 0 0"/>
   </joint>
   <gazebo reference="ft300_sensor">
@@ -421,17 +387,12 @@
     </plugin>
   </gazebo>
-  <gazebo reference="world">
-  </gazebo>
   <gazebo>
     <plugin filename="libgazebo_ros2_control.so" name="gazebo_ros2_control">
       <parameters>/home/lk/ur_sim/src/ur7e_moveit_config/config/ros2_controllers.yaml</parameters>
+      <use_sim_time>true</use_sim_time>   <!-- 关键：为 Gazebo 插件添加仿真时间设置 -->
       <robot_param_node>robot_state_publisher</robot_param_node>
       <robotParam>robot_description</robotParam>
     </plugin>
   </gazebo>
-  <xacro:include filename="$(find realsense2_description)/urdf/_d435i.urdf.xacro" />
-  <xacro:sensor_d435i parent="world" name="camera" use_nominal_extrinsics="true">
-      <origin xyz="0.4 0 2.2" rpy="0 1.5708 0"/>
-  </xacro:sensor_d435i>
   <gazebo reference="camera_link">
       <sensor type="depth" name="d435i_depth_sensor">
